File: hardware/AuraForge_50X - old.kicad_pcb (KiCad board)
At the start: 4 copper layers, 100 x 80 mm, 83 parts, among them J1 TYPE-C-31-M-12, J2 PJ-002AH, J3 PJ-320A, J4 Speaker_Left, J5 Speaker_Right, J6 B2B-XH-A, U1 TPA3116D2DAD, U2 TPS61088RHLR, U3 IP2312-4V35, U4 ESP32-WROOM-32E, U5 DW01A-G, U6 FS8205A, U7 AMS1117-3.3

Commit message: Uploaded all latest files after PCB design update
Parts:
- moved R2 0.81 mm to (105.5, 88.4)
- moved C11 0.51 mm to (158.0, 37.4)
- moved C6 0.21 mm to (102.5, 23.4)
- moved C7 0.21 mm to (102.5, 21.4)
Routing:
- net GND: track 158.9 -> 157.7 mm, vias 366 -> 350
- net Net-(U5-CS): track 4.88 -> 3.78 mm
- net Net-(U1-LINN): track 4.66 -> 3.76 mm
- net /+3V3_SYS: track 233.0 -> 232.1 mm
- net /V_LDO_IN: track 14.2 -> 13.4 mm
- net Net-(J1-CC2): track 6.97 -> 6.27 mm
- net Net-(U2-VCC): track 3.32 -> 2.81 mm
Other:
- board text removed: "AuraForge-50X ============== Ravi Kachhwaha"
