File: hardware/AuraForge_50X.kicad_sch (KiCad schematic)
At the start: 83 parts, among them J1 TYPE-C-31-M-12, J2 PJ-002AH, J3 PJ-320A, J4 Speaker_Left, J5 Speaker_Right, J6 B2B-XH-A, U1 TPA3116D2DAD, U2 TPS61088RHLR, U3 IP2312-4V35, U4 ESP32-WROOM-32E, U5 DW01A-G, U6 FS8205A, U7 AMS1117-3.3

Commit message: Upload updated and fixed files.
Parts:
- R9: value 165k 1% -> 91k 1%
Other:
- company: Hack Club Forge Tier 3 Project -> Hack Club Forge Tier 2 Project
Changed lines of the file:
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@@
 		(date "2026-08-13")
 		(rev "v1.0")
-		(company "Hack Club Forge Tier 3 Project")
+		(company "Hack Club Forge Tier 2 Project")
+		(comment 1 "Ravi Kachhwaha")
 	)
 	(junction
@@
 			)
 		)
-		(property "Value" "165k 1%"
+		(property "Value" "91k 1%"
 			(at 303.784 218.44 90)
 			(show_name no)

Commit message: Uploading latest files of New PCB Layout
Connections:
- net I2S_BCK renamed DAC_OUT_R
- net I2S_LRCK renamed DAC_OUT_L
Changed lines of the file:
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@@
 		)
 	)
-	(label "I2S_BCK"
+	(label "DAC_OUT_R"
 		(at 259.08 142.24 180)
 		(effects
@@
 		)
 	)
-	(label "I2S_LRCK"
+	(label "DAC_OUT_L"
 		(at 48.26 153.67 0)
 		(effects
@@
 		)
 	)
-	(label "I2S_LRCK"
+	(label "DAC_OUT_L"
 		(at 250.19 139.7 180)
 		(effects

Commit message: Latest PCB files uploaded
Parts:
- removed L1: 2.2uH 6.5A, Inductor_SMD:L_7.3x7.3_H4.5, symbol Device:L
- removed L2: 2.2uH 10A, Inductor_SMD:L_10.4x10.4_H4.8, symbol Device:L
- removed L3, L4, L5, L6: 10uH 3.8A, Inductor_SMD:L_Taiyo-Yuden_NR-80xx, symbol Device:L
- added L1: 2.2uH 6.5A, easyeda2kicad:INDM7066X300N, symbol easyeda2kicad:MWSA0603S-2R2MT
- added L2: 2.2uH 10A, easyeda2kicad:WE-HCC_8070, symbol easyeda2kicad:WE-HCC_8070
- added L3, L4, L5, L6: 10uH 3.8A, easyeda2kicad:IND_TAIYO_NRS8040_TAY, symbol easyeda2kicad:NRS8040T100MJGJ
Connections:
- net +BAT_3V7: now also L1.2, L2.1
- net SPK_L_MINUS: now also L4.1
- net SPK_L_PLUS: now also L3.1
- net SPK_R_MINUS: now also L6.1
- net SPK_R_PLUS: now also L5.1
- net at C12.2, U2.4 (SW), U2.5 (SW)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: now also L2.2
- net at C32.2, U1.29 (OUTPR): now also L5.2
- net at C30.2, U1.23 (OUTPL): now also L3.2
- net at U3.7 (SW): now also L1.1
- net at C29.1, U1.21 (OUTNL): now also L4.2
- net at C31.1, U1.27 (OUTNR): now also L6.2

Commit message: Uploaded all latest files after PCB design update
Parts:
- R3: value 45k 1% -> 45.3k 1%
Changed lines of the file:
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@@
 			)
 		)
-		(property "Value" "45k 1%"
+		(property "Value" "45.3k 1%"
 			(at 307.34 44.45 90)
 			(show_name no)
